Commit message: Correct hinge location & turning speed

File: catkin_ws/src/my_robot/urdf/my_robot.xacro (robot description, xacro)
@@ -9,5 +9,5 @@
   </joint>
   <joint type="continuous" name="right_wheel_hinge">
-    <origin xyz="0 0.15 0" rpy="0 0 0"/>
+    <origin xyz="0 -0.15 0" rpy="0 0 0"/>
     <child link="right_wheel"/>
     <parent link="chassis"/>
@@ -17,5 +17,5 @@
   </joint>
   <joint type="continuous" name="left_wheel_hinge">
-    <origin xyz="0 -0.15 0" rpy="0 0 0"/>
+    <origin xyz="0 0.15 0" rpy="0 0 0"/>
     <child link="left_wheel"/>
     <parent link="chassis"/>
